Commit message: add : gazebo simulation

File: src/my_robot_description/urdf/my_robot.urdf (robot description, URDF)
Before this commit: robot simple_diff_drive, 5 links, 4 joints
Links:
- link base_link: mass None -> 0.5; geometry collision box size=0.3 0.2 0.1; visual box size=0.3 0.2 0.1
- link caster_wheel: mass None -> 0.05; geometry collision sphere radius=0.03; visual sphere radius=0.03
- link left_wheel: mass None -> 0.1; geometry collision cylinder length=0.04 radius=0.05; visual cylinder length=0.04 radius=0.05
- link right_wheel: mass None -> 0.1; geometry collision cylinder length=0.04 radius=0.05; visual cylinder length=0.04 radius=0.05

Commit message: add : gazebo laser sensor

File: src/my_robot_description/urdf/my_robot.urdf (robot description, URDF)
Before this commit: robot simple_diff_drive, 5 links, 4 joints
Links:
- added link laser_frame, mass 0.1; collision cylinder length=0.04 radius=0.05; visual cylinder length=0.04 radius=0.05
Joints:
- added joint laser_joint: type fixed, parent base_link, child laser_frame, origin xyz=0.1 0 0.07 rpy=0 0 0
